Commit message: Updated some errors
Co-authored-by: Copilot <copilot@github.com>

File: urdf/cube_robot.xacro (robot description, xacro)
@@ -1,4 +1,10 @@
 <?xml version="1.0"?>
 <robot name="cube_robot" xmlns:xacro="http://www.ros.org/wiki/xacro">
+  <!-- Material definitions -->
+  <material name="blue">
+    <color rgba="0 0 1 1"/>
+  </material>
+  <!-- Dummy root link (workaround for KDL inertia issue) -->
+  <link name="world"/>
   <!-- Base cube -->
   <link name="base_link">
@@ -22,4 +28,9 @@
     </inertial>
   </link>
+  <!-- Joint from world to base_link -->
+  <joint name="world_base_joint" type="fixed">
+    <parent link="world"/>
+    <child link="base_link"/>
+  </joint>
   <!-- Lidar -->
   <link name="lidar_link">
