Commit message: Bridged all gaps

File: urdf/cuboid_robot.urdf.xacro (robot description, xacro)
@@ -1,32 +1,64 @@
 <?xml version="1.0"?>
-<robot xmlns:xacro="http://www.ros.org/wiki/xacro" name="cuboid_robot">
-  <xacro:arg name="use_sim" default="true"/>
+<robot name="cuboid_robot" xmlns:xacro="http://www.ros.org/wiki/xacro">
+  <!-- Base -->
   <link name="base_link">
-    <inertial><origin xyz="0 0 0"/><mass value="20"/><inertia ixx="0.3" ixy="0" ixz="0" iyy="0.8" iyz="0" izz="0.8"/></inertial>
-    <visual><origin xyz="0 0 0"/><geometry><box size="0.6 0.4 0.25"/></geometry><material name="Blue"><color rgba="0.1 0.2 0.8 1.0"/></material></visual>
-    <collision><origin xyz="0 0 0"/><geometry><box size="0.6 0.4 0.25"/></geometry></collision>
+    <visual>
+      <geometry>
+        <box size="0.5 0.3 0.2"/>
+      </geometry>
+    </visual>
+    <collision>
+      <geometry>
+        <box size="0.5 0.3 0.2"/>
+      </geometry>
+    </collision>
+    <inertial>
+      <mass value="5.0"/>
+      <inertia ixx="0.1" iyy="0.1" izz="0.1"
+               ixy="0.0" ixz="0.0" iyz="0.0"/>
+    </inertial>
   </link>
-  <link name="laser_link">
-    <visual><origin xyz="0 0 0"/><geometry><cylinder length="0.03" radius="0.04"/></geometry><material name="Black"><color rgba="0 0 0 1"/></material></visual>
-    <collision><origin xyz="0 0 0"/><geometry><cylinder length="0.03" radius="0.04"/></geometry></collision>
-    <inertial><origin xyz="0 0 0"/><mass value="0.2"/><inertia ixx="0.0002" ixy="0" ixz="0" iyy="0.0002" iyz="0" izz="0.0002"/></inertial>
-  </link>
-  <joint name="laser_joint" type="fixed"><parent link="base_link"/><child link="laser_link"/><origin xyz="0 0 0.145" rpy="0 0 0"/></joint>
-  <link name="base_footprint"/>
-  <joint name="base_footprint_joint" type="fixed"><parent link="base_footprint"/><child link="base_link"/><origin xyz="0 0 0.125" rpy="0 0 0"/></joint>
-  <gazebo>
-    <plugin filename="libgz-sim-pose-publisher-system.so" name="gz::sim::systems::PosePublisher"/>
-  </gazebo>
-  <gazebo reference="base_link">
-    <gravity>true</gravity>
-    <mu1>1.0</mu1><mu2>1.0</mu2>
-  </gazebo>
-  <gazebo reference="laser_link">
+  <!-- Wheels -->
+  <link name="left_wheel"/>
+  <link name="right_wheel"/>
+  <joint name="left_wheel_joint" type="continuous">
+    <parent link="base_link"/>
+    <child link="left_wheel"/>
+    <origin xyz="0 0.2 -0.1"/>
+    <axis xyz="0 1 0"/>
+  </joint>
+  <joint name="right_wheel_joint" type="continuous">
+    <parent link="base_link"/>
+    <child link="right_wheel"/>
+    <origin xyz="0 -0.2 -0.1"/>
+    <axis xyz="0 1 0"/>
+  </joint>
+  <!-- Lidar -->
+  <link name="lidar_link"/>
+  <joint name="lidar_joint" type="fixed">
+    <parent link="base_link"/>
+    <child link="lidar_link"/>
+    <origin xyz="0 0 0.2"/>
+  </joint>
+  <!-- Gazebo Lidar -->
+  <gazebo reference="lidar_link">
     <sensor name="lidar" type="gpu_lidar">
-      <pose>0 0 0 0 0 0</pose>
-      <always_on>true</always_on><update_rate>15</update_rate><visualize>true</visualize>
-      <topic>/scan</topic>
-      <lidar><scan><horizontal><samples>720</samples><resolution>1</resolution><min_angle>-3.14159</min_angle><max_angle>3.14159</max_angle></horizontal></scan><range><min>0.12</min><max>12.0</max><resolution>0.01</resolution></range></lidar>
+      <update_rate>10</update_rate>
+      <topic>scan</topic>
     </sensor>
   </gazebo>
+  <!-- Diff Drive Plugin (CRITICAL) -->
+  <gazebo>
+    <plugin filename="libgz-sim-diff-drive-system.so"
+            name="gz::sim::systems::DiffDrive">
+      <left_joint>left_wheel_joint</left_joint>
+      <right_joint>right_wheel_joint</right_joint>
+      <wheel_separation>0.4</wheel_separation>
+      <wheel_radius>0.1</wheel_radius>
+      <topic>/cmd_vel</topic>
+      <odom_topic>/odom</odom_topic>
+      <frame_id>odom</frame_id>
+      <child_frame_id>base_link</child_frame_id>
+    </plugin>
+  </gazebo>
 </robot>

Commit message: Codex fixes are in

File: urdf/cuboid_robot.urdf.xacro (robot description, xacro)
@@ -1,12 +1,23 @@
 <?xml version="1.0"?>
 <robot name="cuboid_robot" xmlns:xacro="http://www.ros.org/wiki/xacro">
-  <!-- Base -->
+  <material name="gray">
+    <color rgba="0.6 0.6 0.6 1.0"/>
+  </material>
+  <material name="black">
+    <color rgba="0.1 0.1 0.1 1.0"/>
+  </material>
+  <material name="red">
+    <color rgba="0.9 0.1 0.1 1.0"/>
+  </material>
   <link name="base_link">
     <visual>
+      <origin xyz="0 0 0"/>
       <geometry>
         <box size="0.5 0.3 0.2"/>
       </geometry>
+      <material name="gray"/>
     </visual>
     <collision>
+      <origin xyz="0 0 0"/>
       <geometry>
         <box size="0.5 0.3 0.2"/>
@@ -19,7 +30,44 @@
     </inertial>
   </link>
-  <!-- Wheels -->
-  <link name="left_wheel"/>
-  <link name="right_wheel"/>
+  <link name="left_wheel">
+    <visual>
+      <origin rpy="1.5708 0 0"/>
+      <geometry>
+        <cylinder radius="0.1" length="0.05"/>
+      </geometry>
+      <material name="black"/>
+    </visual>
+    <collision>
+      <origin rpy="1.5708 0 0"/>
+      <geometry>
+        <cylinder radius="0.1" length="0.05"/>
+      </geometry>
+    </collision>
+    <inertial>
+      <mass value="0.5"/>
+      <inertia ixx="0.002" iyy="0.001" izz="0.002"
+               ixy="0.0" ixz="0.0" iyz="0.0"/>
+    </inertial>
+  </link>
+  <link name="right_wheel">
+    <visual>
+      <origin rpy="1.5708 0 0"/>
+      <geometry>
+        <cylinder radius="0.1" length="0.05"/>
+      </geometry>
+      <material name="black"/>
+    </visual>
+    <collision>
+      <origin rpy="1.5708 0 0"/>
+      <geometry>
+        <cylinder radius="0.1" length="0.05"/>
+      </geometry>
+    </collision>
+    <inertial>
+      <mass value="0.5"/>
+      <inertia ixx="0.002" iyy="0.001" izz="0.002"
+               ixy="0.0" ixz="0.0" iyz="0.0"/>
+    </inertial>
+  </link>
   <joint name="left_wheel_joint" type="continuous">
     <parent link="base_link"/>
@@ -34,6 +82,22 @@
     <axis xyz="0 1 0"/>
   </joint>
-  <!-- Lidar -->
-  <link name="lidar_link"/>
+  <link name="lidar_link">
+    <visual>
+      <geometry>
+        <cylinder radius="0.05" length="0.06"/>
+      </geometry>
+      <material name="red"/>
+    </visual>
+    <collision>
+      <geometry>
+        <cylinder radius="0.05" length="0.06"/>
+      </geometry>
+    </collision>
+    <inertial>
+      <mass value="0.1"/>
+      <inertia ixx="0.0002" iyy="0.0002" izz="0.0002"
+               ixy="0.0" ixz="0.0" iyz="0.0"/>
+    </inertial>
+  </link>
   <joint name="lidar_joint" type="fixed">
     <parent link="base_link"/>
@@ -41,12 +105,26 @@
     <origin xyz="0 0 0.2"/>
   </joint>
-  <!-- Gazebo Lidar -->
   <gazebo reference="lidar_link">
     <sensor name="lidar" type="gpu_lidar">
       <update_rate>10</update_rate>
-      <topic>scan</topic>
+      <topic>/scan</topic>
+      <gz_frame_id>lidar_link</gz_frame_id>
+      <lidar>
+        <scan>
+          <horizontal>
+            <samples>360</samples>
+            <resolution>1</resolution>
+            <min_angle>-3.14159</min_angle>
+            <max_angle>3.14159</max_angle>
+          </horizontal>
+        </scan>
+        <range>
+          <min>0.12</min>
+          <max>12.0</max>
+          <resolution>0.01</resolution>
+        </range>
+      </lidar>
     </sensor>
   </gazebo>
-  <!-- Diff Drive Plugin (CRITICAL) -->
   <gazebo>
     <plugin filename="libgz-sim-diff-drive-system.so"

Commit message: Fix

File: urdf/cuboid_robot.urdf.xacro (robot description, xacro)
@@ -84,12 +84,14 @@
   <link name="lidar_link">
     <visual>
+      <origin xyz="0 0 0.03"/>
       <geometry>
-        <cylinder radius="0.05" length="0.06"/>
+        <cylinder radius="0.06" length="0.06"/>
       </geometry>
       <material name="red"/>
     </visual>
     <collision>
+      <origin xyz="0 0 0.03"/>
       <geometry>
-        <cylinder radius="0.05" length="0.06"/>
+        <cylinder radius="0.06" length="0.06"/>
       </geometry>
     </collision>
@@ -103,12 +105,14 @@
     <parent link="base_link"/>
     <child link="lidar_link"/>
-    <origin xyz="0 0 0.2"/>
+    <origin xyz="0 0 0.16"/>
   </joint>
   <gazebo reference="lidar_link">
-    <sensor name="lidar" type="gpu_lidar">
+    <sensor name="lidar" type="ray">
+      <pose>0 0 0 0 0 0</pose>
+      <visualize>true</visualize>
       <update_rate>10</update_rate>
       <topic>/scan</topic>
       <gz_frame_id>lidar_link</gz_frame_id>
-      <lidar>
+      <ray>
         <scan>
           <horizontal>
@@ -124,5 +128,5 @@
           <resolution>0.01</resolution>
         </range>
-      </lidar>
+      </ray>
     </sensor>
   </gazebo>

Commit message: Some extra fixes

File: urdf/cuboid_robot.urdf.xacro (robot description, xacro)
@@ -70,15 +70,13 @@
     </inertial>
   </link>
-  <joint name="left_wheel_joint" type="continuous">
+  <joint name="left_wheel_joint" type="fixed">
     <parent link="base_link"/>
     <child link="left_wheel"/>
     <origin xyz="0 0.2 -0.1"/>
-    <axis xyz="0 1 0"/>
   </joint>
-  <joint name="right_wheel_joint" type="continuous">
+  <joint name="right_wheel_joint" type="fixed">
     <parent link="base_link"/>
     <child link="right_wheel"/>
     <origin xyz="0 -0.2 -0.1"/>
-    <axis xyz="0 1 0"/>
   </joint>
   <link name="lidar_link">
